File: hardware/PSU/PSU.kicad_sch (KiCad schematic)
At the start: 0 parts

Commit message: Initial schematic
Parts:
- added C1: 100uF 50v, Capacitor_SMD:CP_Elec_6.3x7.7, symbol Device:C_Polarized_Small
- added C2, C3: 10uF 50v, Capacitor_SMD:CP_Elec_5x5.4, symbol Device:C_Polarized_Small
- added C4, C5: 22uF 25v, Capacitor_SMD:CP_Elec_5x5.4, symbol Device:C_Polarized_Small
- added C6, C7: 4.7uF 25v, Capacitor_SMD:C_0805_2012Metric_Pad1.18x1.45mm_HandSolder, symbol Device:C_Small
- added CN1, CN2: JST PH 2 pin male, easyeda2kicad:CONN-TH_B2B-PH-K-S, symbol easyeda2kicad:B2B-PH-K-S(LF)(SN)
- added D1: Barrier, Diode_SMD:D_SMA_Handsoldering, symbol Device:D_Schottky_Small
- added D2, D3, D4: LED, LED_SMD:LED_0805_2012Metric_Pad1.15x1.40mm_HandSolder, symbol Device:LED
- added F1: 1.5A 24V, Fuse:Fuse_1812_4532Metric_Pad1.30x3.40mm_HandSolder, symbol Device:Fuse_Small
- added H1, H2, H3, H4: ~, MountingHole:MountingHole_3.2mm_M3_Pad, symbol Mechanical:MountingHole_Pad
- added J1, J2: IDC 2x5 male, Connector_IDC:IDC-Header_2x05_P2.54mm_Vertical, symbol Connector_Generic:Conn_02x05_Odd_Even
- added L1: 10uH 800mA, symbol Device:L
- added R1, R2, R3: 5.1k, Resistor_SMD:R_0805_2012Metric_Pad1.20x1.40mm_HandSolder, symbol Device:R_Small
- added RV1: MOV 18v, Resistor_SMD:R_1206_3216Metric_Pad1.30x1.75mm_HandSolder, symbol Device:Varistor
- added U1, U2: K7812-1000R3, easyeda2kicad:PWRM-TH_K7812-1000R3, symbol easyeda2kicad:K7812-1000R3_C5369648
Connections:
- new net: D4.1 (K), R3.1
- new net: D3.1 (K), R2.2
- new net: C3.1, L1.2, U2.1 (Vin)
- new net: D1.1 (K), F1.1
- new net: D2.1 (K), R1.1
- new net +12V: C5.1, C6.1, D2.2 (A), J1.10 (Pin_10), J1.9 (Pin_9), J2.10 (Pin_10), J2.9 (Pin_9), U1.3 (+Vo/GND)
- new net +15V: C1.1, C2.1, D4.2 (A), F1.2, L1.1, RV1.1, U1.1 (Vin)
- new net -12V: C4.1, C7.1, J1.1 (Pin_1), J1.2 (Pin_2), J2.1 (Pin_1), J2.2 (Pin_2), R2.1, U2.2 (GND/-Vo)
- new net GND: C1.2, C2.2, C3.2, C4.2, C5.2, C6.2, C7.2, CN1.2, CN2.2, D3.2 (A), H1.1, H2.1, H3.1, H4.1, J1.3 (Pin_3), J1.4 (Pin_4), J1.5 (Pin_5), J1.6 (Pin_6), J1.7 (Pin_7), J1.8 (Pin_8), J2.3 (Pin_3), J2.4 (Pin_4), J2.5 (Pin_5), J2.6 (Pin_6), J2.7 (Pin_7), J2.8 (Pin_8), R1.2, R3.2, RV1.2, U1.2 (GND/-Vo), U2.3 (+Vo/GND)
- new net VIN: CN1.1, CN2.1, D1.2 (A)
Other:
- note added: "Circuit protection"
- note added: "DC input"
- note added: "Eurorack power"
- note added: "Mounting holes"
- note added: "Power Indicators"
- note added: "Power conversion"

Commit message: Initial board layout
Parts:
- L1: footprint (none) -> PSU_Parts:L_muRata_LQH3NPZ100MMEL_HandSolder
Changed lines of the file:
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@@
 			)
 		)
-		(property "Footprint" ""
+		(property "Footprint" "PSU_Parts:L_muRata_LQH3NPZ100MMEL_HandSolder"
 			(at 45.72 130.81 0)
 			(effects

Commit message: Add test points
Parts:
- added TP1, TP2: GND, TestPoint:TestPoint_Keystone_5000-5004_Miniature, symbol Connector:TestPoint
- added TP3: +12v, TestPoint:TestPoint_Keystone_5000-5004_Miniature, symbol Connector:TestPoint
- added TP4: -12v, TestPoint:TestPoint_Keystone_5000-5004_Miniature, symbol Connector:TestPoint
- added TP5: +15v, TestPoint:TestPoint_Keystone_5000-5004_Miniature, symbol Connector:TestPoint
Connections:
- net +12V: now also TP3.1
- net +15V: now also TP5.1
- net -12V: now also C4.2, C7.2, TP4.1; no longer C4.1, C7.1
- net GND: now also C4.1, C7.1, TP1.1, TP2.1; no longer C4.2, C7.2
Other:
- note added: "Test points"
- moved on the sheet: C4, C7

Commit message: Use 3mm LEDs instead
Parts:
- D2, D3, D4: footprint LED_SMD:LED_0805_2012Metric_Pad1.15x1.40mm_HandSolder -> LED_THT:LED_D3.0mm
Changed lines of the file:
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@@
 			)
 		)
-		(property "Footprint" "LED_SMD:LED_0805_2012Metric_Pad1.15x1.40mm_HandSolder"
+		(property "Footprint" "LED_THT:LED_D3.0mm"
 			(at 124.46 40.64 0)
 			(effects
@@
 			)
 		)
-		(property "Footprint" "LED_SMD:LED_0805_2012Metric_Pad1.15x1.40mm_HandSolder"
+		(property "Footprint" "LED_THT:LED_D3.0mm"
 			(at 107.95 53.34 0)
 			(effects
@@
 			)
 		)
-		(property "Footprint" "LED_SMD:LED_0805_2012Metric_Pad1.15x1.40mm_HandSolder"
+		(property "Footprint" "LED_THT:LED_D3.0mm"
 			(at 91.44 40.64 0)
 			(effects
