File: hardware/faceplate/faceplate.kicad_pcb (KiCad board)
At the start: 2 copper layers, 30 x 128.5 mm, 11 parts

Commit message: Update faceplate and hit print
Parts:
- REF** (x7): value MountingHole_3.2mm_M3 -> MountingHole_3.2mm_M3_naked; footprint MountingHole:MountingHole_3.2mm_M3 -> ModularMountingHoles:MountingHole_3.2mm_M3_naked
Other:
- board text added: "+12V"
- board text added: "+15V"
- board text added: "-12V"
Changed lines of the file:
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@@
 	)
 	(net 0 "")
-	(footprint "MountingHole:MountingHole_3.2mm_M3"
+	(footprint "ModularMountingHoles:MountingHole_3.2mm_M3_naked"
 		(layer "F.Cu")
 		(at 75 88.58)
@@
 			)
 		)
-		(property "Value" "MountingHole_3.2mm_M3"
+		(property "Value" "MountingHole_3.2mm_M3_naked"
 			(at 0 4.15 0)
 			(layer "F.Fab")
@@
 		)
 		(attr exclude_from_pos_files exclude_from_bom)
-		(fp_circle
-			(center 0 0)
-			(end 3.2 0)
-			(stroke
-				(width 0.15)
-				(type solid)
-			)
-			(fill no)
-			(layer "Cmts.User")
-		)
-		(fp_circle
-			(center 0 0)
-			(end 3.45 0)
-			(stroke
-				(width 0.05)
-				(type solid)
-			)
-			(fill no)
-			(layer "F.CrtYd")
-		)
 		(pad "" np_thru_hole circle
 			(at 0 0)
@@
 		(embedded_fonts no)
 	)
-	(footprint "MountingHole:MountingHole_3.2mm_M3"
+	(footprint "ModularMountingHoles:MountingHole_3.2mm_M3_naked"
 		(layer "F.Cu")
 		(at 75 63.25)
@@
 			)
 		)
-		(property "Value" "MountingHole_3.2mm_M3"
+		(property "Value" "MountingHole_3.2mm_M3_naked"
 			(at 0 4.15 0)
 			(layer "F.Fab")
@@
 		)
 		(attr exclude_from_pos_files exclude_from_bom)
-		(fp_circle
-			(center 0 0)
-			(end 3.2 0)
-			(stroke
-				(width 0.15)
-				(type solid)
-			)
-			(fill no)
-			(layer "Cmts.User")
-		)
-		(fp_circle
-			(center 0 0)
-			(end 3.45 0)
-			(stroke
-				(width 0.05)
-				(type solid)
-			)
-			(fill no)
-			(layer "F.CrtYd")
-		)
 		(pad "" np_thru_hole circle
 			(at 0 0)
@@
 		(embedded_fonts no)
 	)
-	(footprint "MountingHole:MountingHole_3.2mm_M3"
+	(footprint "ModularMountingHoles:MountingHole_3.2mm_M3_naked"
 		(layer "F.Cu")
 		(at 55 63.25)
@@
 			)
 		)
-		(property "Value" "MountingHole_3.2mm_M3"
+		(property "Value" "MountingHole_3.2mm_M3_naked"
 			(at 0 4.15 0)
 			(layer "F.Fab")
@@
 		)
 		(attr exclude_from_pos_files exclude_from_bom)
-		(fp_circle
-			(center 0 0)
-			(end 3.2 0)
-			(stroke
-				(width 0.15)
-				(type solid)
-			)
-			(fill no)
-			(layer "Cmts.User")
-		)
-		(fp_circle
-			(center 0 0)
-			(end 3.45 0)
-			(stroke
-				(width 0.05)
-				(type solid)
-			)
-			(fill no)
-			(layer "F.CrtYd")
-		)
 		(pad "" np_thru_hole circle
 			(at 0 0)
@@
 		(embedded_fonts no)
 	)
-	(footprint "MountingHole:MountingHole_3.2mm_M3"
+	(footprint "ModularMountingHoles:MountingHole_3.2mm_M3_naked"
 		(layer "F.Cu")
 		(at 75 165.25)
@@
 			)
 		)
-		(property "Value" "MountingHole_3.2mm_M3"
+		(property "Value" "MountingHole_3.2mm_M3_naked"
 			(at 0 4.15 0)
 			(layer "F.Fab")
@@
 		)
 		(attr exclude_from_pos_files exclude_from_bom)
-		(fp_circle
-			(center 0 0)
-			(end 3.2 0)
-			(stroke
-				(width 0.15)
-				(type solid)
-			)
-			(fill no)
-			(layer "Cmts.User")
-		)
-		(fp_circle
-			(center 0 0)
-			(end 3.45 0)
-			(stroke
-				(width 0.05)
-				(type solid)
-			)
-			(fill no)
-			(layer "F.CrtYd")
-		)
 		(pad "" np_thru_hole circle
 			(at 0 0)
@@
 		(embedded_fonts no)
 	)
-	(footprint "MountingHole:MountingHole_3.2mm_M3"
+	(footprint "ModularMountingHoles:MountingHole_3.2mm_M3_naked"
 		(layer "F.Cu")
 		(at 75 98.58)
@@
 			)
 		)
-		(property "Value" "MountingHole_3.2mm_M3"
+		(property "Value" "MountingHole_3.2mm_M3_naked"
 			(at 0 4.15 0)
 			(layer "F.Fab")
@@
 		)
 		(attr exclude_from_pos_files exclude_from_bom)
-		(fp_circle
-			(center 0 0)
-			(end 3.2 0)
-			(stroke
-				(width 0.15)
-				(type solid)
-			)
-			(fill no)
-			(layer "Cmts.User")
-		)
-		(fp_circle
-			(center 0 0)
-			(end 3.45 0)
-			(stroke
-				(width 0.05)
-				(type solid)
-			)
-			(fill no)
-			(layer "F.CrtYd")
-		)
 		(pad "" np_thru_hole circle
 			(at 0 0)
@@
 		(embedded_fonts no)
 	)
-	(footprint "MountingHole:MountingHole_3.2mm_M3"
+	(footprint "ModularMountingHoles:MountingHole_3.2mm_M3_naked"
 		(layer "F.Cu")
 		(at 75 93.58)
@@
 			)
 		)
-		(property "Value" "MountingHole_3.2mm_M3"
+		(property "Value" "MountingHole_3.2mm_M3_naked"
 			(at 0 4.15 0)
 			(layer "F.Fab")
@@
 		)
 		(attr exclude_from_pos_files exclude_from_bom)
-		(fp_circle
-			(center 0 0)
-			(end 3.2 0)
-			(stroke
-				(width 0.15)
-				(type solid)
-			)
-			(fill no)
-			(layer "Cmts.User")
-		)
-		(fp_circle
-			(center 0 0)
-			(end 3.45 0)
-			(stroke
-				(width 0.05)
-				(type solid)
-			)
-			(fill no)
-			(layer "F.CrtYd")
-		)
 		(pad "" np_thru_hole circle
 			(at 0 0)
@@
 		(embedded_fonts no)
 	)
-	(footprint "MountingHole:MountingHole_3.2mm_M3"
+	(footprint "ModularMountingHoles:MountingHole_3.2mm_M3_naked"
 		(layer "F.Cu")
 		(at 55 165.25)
@@
 			)
 		)
-		(property "Value" "MountingHole_3.2mm_M3"
+		(property "Value" "MountingHole_3.2mm_M3_naked"
 			(at 0 4.15 0)
 			(layer "F.Fab")
@@
 		)
 		(attr exclude_from_pos_files exclude_from_bom)
-		(fp_circle
-			(center 0 0)
-			(end 3.2 0)
-			(stroke
-				(width 0.15)
-				(type solid)
-			)
-			(fill no)
-			(layer "Cmts.User")
-		)
-		(fp_circle
-			(center 0 0)
-			(end 3.45 0)
-			(stroke
-				(width 0.05)
-				(type solid)
-			)
-			(fill no)
-			(layer "F.CrtYd")
-		)
 		(pad "" np_thru_hole circle
 			(at 0 0)
@@
 		(layer "Edge.Cuts")
 	)
+	(gr_text "+15V"
+		(at 73 90 0)
+		(layer "F.SilkS")
+		(effects
+			(font
+				(size 2 2)
+				(thickness 0.25)
+			)
+			(justify right bottom)
+		)
+	)
+	(gr_text "+12V"
+		(at 73 95 0)
+		(layer "F.SilkS")
+		(effects
+			(font
+				(size 2 2)
+				(thickness 0.25)
+			)
+			(justify right bottom)
+		)
+	)
+	(gr_text "-12V"
+		(at 73 100 0)
+		(layer "F.SilkS")
+		(effects
+			(font
+				(size 2 2)
+				(thickness 0.25)
+			)
+			(justify right bottom)
+		)
+	)
 	(embedded_fonts no)
